Commit message: created core URDF

File: description/robot_core.xacro (robot description, xacro)
@@ -25,5 +25,5 @@
     <link name="chassis">
         <visual>
-            <origin xyz="0.15 0 0.75"/>
+            <origin xyz="0.15 0 0.075"/>
             <geometry>
                 <box size="0.3 0.3 0.15"/>
@@ -32,5 +32,5 @@
         </visual>
         <collision>
-            <origin xyz="0.15 0 0.75"/>
+            <origin xyz="0.15 0 0.075"/>
             <geometry>
                 <box size="0.3 0.3 0.15"/>

Commit message: created core URDF

File: description/robot_core.xacro (robot description, xacro)
@@ -41,4 +41,7 @@
         </xacro:inertial_box>
     </link>
+    <gazebo reference="chassis">
+        <material>Gazebo/white</material>
+    </gazebo>
 <!-- LEFT WHEEL LINK-->
     <joint name="left_wheel_joint" type="continuous">
@@ -64,4 +67,7 @@
         </xacro:inertial_cylinder>
     </link>
+    <gazebo reference="left_wheel">
+        <material>Gazebo/Blue</material>
+    </gazebo>
 <!-- RIGHT WHEEL LINK-->
     <joint name="right_wheel_joint" type="continuous">
@@ -88,4 +94,7 @@
         </xacro:inertial_cylinder>
     </link>
+    <gazebo reference="right_wheel">
+        <material>Gazebo/Blue</material>
+    </gazebo>
 <!--CASTOR WHEEL LINK-->
     <joint name="castor_wheel_joint" type="fixed">
@@ -111,3 +120,8 @@
         </xacro:inertial_sphere>
     </link>
+    <gazebo reference="castor_wheel">
+        <material>Gazebo/Black</material>
+        <mu1 value ="0.001"/>
+        <mu1 value ="0.001"/>
+    </gazebo>
 </robot>
